File: DISPLAY.sch (KiCad schematic (older format))
At the start: 3 parts, among them U10 MCP23008-xP

Commit message: ported over LCD display code, modified schematic as we no longer need some of the I2C expanders
Parts:
- added RV1: 10K LIN, symbol Device:R_POT
- U10: footprint Package_DIP:DIP-18_W7.62mm -> (none)
Connections:
- wire segments 53 -> 56
Other:
- note removed: "TODO!!!"
Changed lines of the file:
@@
 U 1 1 6096E5BE
 P 6500 3100
-F 0 "DS1" H 6900 4100 50  0000 C CNN
-F 1 "16x02 LCD display WC1602A" H 7350 4000 50  0000 C CNN
+F 0 "DS1" V 7000 2650 50  0000 C CNN
+F 1 "16x02 LCD display WC1602A" V 7100 2650 50  0000 C CNN
 F 2 "Display:WC1602A" H 6500 2200 50  0001 C CIN
 F 3 "http://www.wincomlcd.com/pdf/WC1602A-SFYLYHTC06.pdf" H 7200 3100 50  0001 C CNN
@@
 	1    0    0    -1
 $EndComp
-Wire Wire Line
-	6500 2200 6500 2300
 $Comp
 L Interface_Expansion:MCP23008-xP U?
@@
 AR Path="/604E5285/5FEF98BC" Ref="U?"  Part="1"
 AR Path="/6096B205/5FEF98BC" Ref="U10"  Part="1"
-F 0 "U10" V 5050 3600 50  0000 C CNN
-F 1 "MCP23008-xP" V 5200 3650 50  0000 C CNN
-F 2 "Package_DIP:DIP-18_W7.62mm" H 5050 2550 50  0001 C CNN
+F 0 "U10" V 5000 3600 50  0000 C CNN
+F 1 "MCP23008-xP" V 5100 3600 50  0000 C CNN
+F 2 "" H 5050 2550 50  0001 C CNN
 F 3 "http://ww1.microchip.com/downloads/en/DeviceDoc/MCP23008-MCP23S08-Data-Sheet-20001919F.pdf" H 6350 2400 50  0001 C CNN
 	1    5050 3600
@@
 $EndComp
 Wire Wire Line
-	7300 2900 7300 4300
-Wire Wire Line
-	7300 4300 6500 4300
-Wire Wire Line
-	6900 2900 7300 2900
-Connection ~ 6500 4300
-Wire Wire Line
-	6900 2800 7300 2800
-Text Notes 7350 2650 0    50   ~ 0
-TODO!!!
-Wire Wire Line
 	6100 2500 5850 2500
 Wire Wire Line
@@
 Text GLabel 5850 2700 0    50   Input ~ 0
 LCD_REGSEL
-Wire Wire Line
-	6900 2500 7300 2500
 Wire Wire Line
 	5050 4300 5750 4300
@@
 	4300 3850 4300 3900
 Connection ~ 4300 3900
+$Comp
+L Device:R_POT RV1
+U 1 1 5FF69F75
+P 7450 2500
+F 0 "RV1" H 7380 2454 50  0000 R CNN
+F 1 "10K LIN" H 7380 2545 50  0000 R CNN
+F 2 "" H 7450 2500 50  0001 C CNN
+F 3 "~" H 7450 2500 50  0001 C CNN
+	1    7450 2500
+	-1   0    0    1
+$EndComp
+$Comp
+L power:+3V3 #PWR?
+U 1 1 5FF6DEDA
+P 7100 2750
+AR Path="/604E5285/5FF6DEDA" Ref="#PWR?"  Part="1"
+AR Path="/6096B205/5FF6DEDA" Ref="#PWR0116"  Part="1"
+F 0 "#PWR0116" H 7100 2600 50  0001 C CNN
+F 1 "+3V3" H 7115 2923 50  0000 C CNN
+F 2 "" H 7100 2750 50  0001 C CNN
+F 3 "" H 7100 2750 50  0001 C CNN
+	1    7100 2750
+	1    0    0    -1
+$EndComp
+Wire Wire Line
+	7450 2350 7450 2250
+Wire Wire Line
+	6900 2800 7100 2800
+Wire Wire Line
+	7100 2800 7100 2750
+Wire Wire Line
+	6500 2200 6500 2250
+Wire Wire Line
+	7450 2650 7450 4300
+Wire Wire Line
+	6900 2500 7300 2500
+Wire Wire Line
+	7450 2250 6500 2250
+Connection ~ 6500 2250
+Wire Wire Line
+	6500 2250 6500 2300
+Wire Wire Line
+	7400 4300 6500 4300
+Connection ~ 6500 4300
 $EndSCHEMATC
