File: DISPLAY.sch (KiCad schematic (older format))
At the start: 4 parts, among them U10 MCP23008-xP

Commit message: Replaced digital pots with analog, removed spi bus too as no longer needed
Parts:
- removed C17: 0.1uF, symbol Device:C
- removed DS1: 16x02 LCD display WC1602A, Display:WC1602A, symbol Display_Character:WC1602A
- removed RV1: 10K LIN, symbol Device:R_POT
- removed U10: MCP23008-xP, symbol Interface_Expansion:MCP23008-xP
Connections:
- net labels removed: +3V3, GND, I2C_SCL, I2C_SDA, LCD_ENABLE, LCD_REGSEL, LCD_RW, RESET
- wire segments 56 -> 0
- no-connect marks 1 -> 0
