File: PSUs.sch (KiCad schematic (older format))
At the start: 41 parts, among them Q1 2N2222, Q2 2N2222, U1 LM2674N-ADJ, U2 LM2574N-3.3, U3 LM2674N-ADJ, U4 LM2674N-5.0

Commit message: replaced capacitor multiplier by using a more powerful output transistor
Parts:
- removed C7, C8: 10uF 25V, symbol Device:CP
- C5, C6: value 10uF 25V -> 470uF 25V
- Q1, Q2: value 2N2222 -> BD139
- R8, R9: value 10K -> 1K
Connections:
- wire segments 166 -> 158
Changed lines of the file:
@@
 VIN
 Wire Wire Line
-	2300 6250 2300 6400
+	3900 6250 3900 6400
 $Comp
 L power:GND #PWR?
 U 1 1 605245B5
-P 2300 6400
+P 3900 6400
 AR Path="/605245B5" Ref="#PWR?"  Part="1"
 AR Path="/604D3BA3/605245B5" Ref="#PWR0101"  Part="1"
-F 0 "#PWR0101" H 2300 6150 50  0001 C CNN
-F 1 "GND" H 2305 6227 50  0000 C CNN
-F 2 "" H 2300 6400 50  0001 C CNN
-F 3 "" H 2300 6400 50  0001 C CNN
-	1    2300 6400
+F 0 "#PWR0101" H 3900 6150 50  0001 C CNN
+F 1 "GND" H 3905 6227 50  0000 C CNN
+F 2 "" H 3900 6400 50  0001 C CNN
+F 3 "" H 3900 6400 50  0001 C CNN
+	1    3900 6400
 	1    0    0    -1
 $EndComp
@@
 L power:GND #PWR?
 U 1 1 60524625
-P 2300 3550
+P 3900 3550
 AR Path="/60524625" Ref="#PWR?"  Part="1"
 AR Path="/604D3BA3/60524625" Ref="#PWR0104"  Part="1"
-F 0 "#PWR0104" H 2300 3300 50  0001 C CNN
-F 1 "GND" H 2305 3377 50  0000 C CNN
-F 2 "" H 2300 3550 50  0001 C CNN
-F 3 "" H 2300 3550 50  0001 C CNN
-	1    2300 3550
-	1    0    0    -1
-$EndComp
-Wire Wire Line
-	2300 3400 2300 3500
+F 0 "#PWR0104" H 3900 3300 50  0001 C CNN
+F 1 "GND" H 3905 3377 50  0000 C CNN
+F 2 "" H 3900 3550 50  0001 C CNN
+F 3 "" H 3900 3550 50  0001 C CNN
+	1    3900 3550
+	1    0    0    -1
+$EndComp
+Wire Wire Line
+	3900 3400 3900 3500
 Text GLabel 1250 2400 0    50   Input ~ 0
 VIN
@@
 L power:PWR_FLAG #FLG0101
 U 1 1 5FF5E115
-P 2300 3500
-F 0 "#FLG0101" H 2300 3575 50  0001 C CNN
-F 1 "PWR_FLAG" V 2300 3628 50  0000 L CNN
-F 2 "" H 2300 3500 50  0001 C CNN
-F 3 "~" H 2300 3500 50  0001 C CNN
-	1    2300 3500
-	0    1    1    0
-$EndComp
-Connection ~ 2300 3500
-Wire Wire Line
-	2300 3500 2300 3550
+P 3900 3500
+F 0 "#FLG0101" H 3900 3575 50  0001 C CNN
+F 1 "PWR_FLAG" V 3900 3628 50  0000 L CNN
+F 2 "" H 3900 3500 50  0001 C CNN
+F 3 "~" H 3900 3500 50  0001 C CNN
+	1    3900 3500
+	0    1    1    0
+$EndComp
+Connection ~ 3900 3500
+Wire Wire Line
+	3900 3500 3900 3550
 $Comp
 L Device:R R4
@@
 P 5150 2800
 F 0 "R8" V 4943 2800 50  0000 C CNN
-F 1 "10K" V 5034 2800 50  0000 C CNN
+F 1 "1K" V 5034 2800 50  0000 C CNN
 F 2 "" V 5080 2800 50  0001 C CNN
 F 3 "~" H 5150 2800 50  0001 C CNN
@@
 AR Path="/604D3BA3/5FFB3873" Ref="C5"  Part="1"
 F 0 "C5" H 5568 3146 50  0000 L CNN
-F 1 "10uF 25V" H 5568 3055 50  0000 L CNN
+F 1 "470uF 25V" H 5568 3055 50  0000 L CNN
 F 2 "" H 5488 2950 50  0001 C CNN
 F 3 "~" H 5450 3100 50  0001 C CNN
@@
 P 5800 2550
 F 0 "Q1" V 6128 2550 50  0000 C CNN
-F 1 "2N2222" V 6037 2550 50  0000 C CNN
+F 1 "BD139" V 6037 2550 50  0000 C CNN
 F 2 "Package_TO_SOT_THT:TO-39-3" H 6000 2475 50  0001 L CIN
 F 3 "http://www.onsemi.com/pub_link/Collateral/2N2219-D.PDF" H 5800 2550 50  0001 L CNN
@@
 Wire Wire Line
 	4400 2800 4800 2800
-$Comp
-L Device:CP C?
-U 1 1 5FFDA7AB
-P 6100 3100
-AR Path="/5FFDA7AB" Ref="C?"  Part="1"
-AR Path="/604D3BA3/5FFDA7AB" Ref="C7"  Part="1"
-F 0 "C7" H 6218 3146 50  0000 L CNN
-F 1 "10uF 25V" H 6218 3055 50  0000 L CNN
-F 2 "" H 6138 2950 50  0001 C CNN
-F 3 "~" H 6100 3100 50  0001 C CNN
-	1    6100 3100
-	1    0    0    -1
-$EndComp
-Wire Wire Line
-	6000 2450 6100 2450
-Wire Wire Line
-	6100 2450 6100 2950
-Wire Wire Line
-	5450 3400 6100 3400
-Wire Wire Line
-	6100 3400 6100 3250
-Connection ~ 5450 3400
-Wire Wire Line
-	6100 2450 6450 2450
 Wire Wire Line
 	6450 2450 6450 2150
-Connection ~ 6100 2450
 $Comp
 L Device:R R9
@@
 P 5150 5650
 F 0 "R9" V 4943 5650 50  0000 C CNN
-F 1 "10K" V 5034 5650 50  0000 C CNN
+F 1 "1K" V 5034 5650 50  0000 C CNN
 F 2 "" V 5080 5650 50  0001 C CNN
 F 3 "~" H 5150 5650 50  0001 C CNN
@@
 AR Path="/604D3BA3/60043E6E" Ref="C6"  Part="1"
 F 0 "C6" H 5568 5996 50  0000 L CNN
-F 1 "10uF 25V" H 5568 5905 50  0000 L CNN
+F 1 "470uF 25V" H 5568 5905 50  0000 L CNN
 F 2 "" H 5488 5800 50  0001 C CNN
 F 3 "~" H 5450 5950 50  0001 C CNN
@@
 P 5800 5400
 F 0 "Q2" V 6128 5400 50  0000 C CNN
-F 1 "2N2222" V 6037 5400 50  0000 C CNN
+F 1 "BD139" V 6037 5400 50  0000 C CNN
 F 2 "Package_TO_SOT_THT:TO-39-3" H 6000 5325 50  0001 L CIN
 F 3 "http://www.onsemi.com/pub_link/Collateral/2N2219-D.PDF" H 5800 5400 50  0001 L CNN
@@
 Wire Wire Line
 	4400 5650 4800 5650
-$Comp
-L Device:CP C?
-U 1 1 60043E8E
-P 6100 5950
-AR Path="/60043E8E" Ref="C?"  Part="1"
-AR Path="/604D3BA3/60043E8E" Ref="C8"  Part="1"
-F 0 "C8" H 6218 5996 50  0000 L CNN
-F 1 "10uF 25V" H 6218 5905 50  0000 L CNN
-F 2 "" H 6138 5800 50  0001 C CNN
-F 3 "~" H 6100 5950 50  0001 C CNN
-	1    6100 5950
-	1    0    0    -1
-$EndComp
-Wire Wire Line
-	6000 5300 6100 5300
-Wire Wire Line
-	6100 5300 6100 5800
-Wire Wire Line
-	5450 6250 6100 6250
-Wire Wire Line
-	6100 6250 6100 6100
-Connection ~ 5450 6250
-Wire Wire Line
-	6100 5300 6450 5300
 Wire Wire Line
 	6450 5300 6450 5000
-Connection ~ 6100 5300
 Connection ~ 3900 6250
 Wire Wire Line
@@
 Text Notes 6950 2950 0    50   ~ 0
 8-40Vin
+Wire Wire Line
+	6000 2450 6450 2450
+Wire Wire Line
+	6000 5300 6450 5300
 $EndSCHEMATC

Commit message: fixed error in schematic after building up parts of circuit
Parts:
- removed C2, C4: 10uF 25V, symbol Device:CP
Connections:
- wire segments 158 -> 148
Changed lines of the file:
@@
 	0    1    1    0
 $EndComp
-$Comp
-L Device:CP COUT?
-U 1 1 5FFA3978
-P 4800 3100
-AR Path="/5FFA3978" Ref="COUT?"  Part="1"
-AR Path="/604D3BA3/5FFA3978" Ref="C2"  Part="1"
-F 0 "C2" H 4918 3146 50  0000 L CNN
-F 1 "10uF 25V" H 4918 3055 50  0000 L CNN
-F 2 "" H 4838 2950 50  0001 C CNN
-F 3 "~" H 4800 3100 50  0001 C CNN
-	1    4800 3100
-	1    0    0    -1
-$EndComp
-Wire Wire Line
-	4800 2800 4800 2950
 Wire Wire Line
 	3900 2800 4400 2800
-Wire Wire Line
-	4800 3250 4800 3400
-Wire Wire Line
-	4800 3400 3900 3400
 Connection ~ 3900 3400
 $Comp
@@
 $EndComp
 Wire Wire Line
-	4800 2800 5000 2800
-Connection ~ 4800 2800
-Wire Wire Line
 	5300 2800 5450 2800
 Wire Wire Line
@@
 Wire Wire Line
 	5450 3250 5450 3400
-Wire Wire Line
-	5450 3400 4800 3400
-Connection ~ 4800 3400
 Connection ~ 5450 2800
 $Comp
@@
 Connection ~ 4400 2800
 Wire Wire Line
-	4400 2800 4800 2800
-Wire Wire Line
 	6450 2450 6450 2150
 $Comp
@@
 	0    1    1    0
 $EndComp
-$Comp
-L Device:CP C?
-U 1 1 60043E61
-P 4800 5950
-AR Path="/60043E61" Ref="C?"  Part="1"
-AR Path="/604D3BA3/60043E61" Ref="C4"  Part="1"
-F 0 "C4" H 4918 5996 50  0000 L CNN
-F 1 "10uF 25V" H 4918 5905 50  0000 L CNN
-F 2 "" H 4838 5800 50  0001 C CNN
-F 3 "~" H 4800 5950 50  0001 C CNN
-	1    4800 5950
-	1    0    0    -1
-$EndComp
-Wire Wire Line
-	4800 5650 4800 5800
-Wire Wire Line
-	4800 6100 4800 6250
-Wire Wire Line
-	4800 6250 3900 6250
 $Comp
 L Device:CP C?
@@
 $EndComp
 Wire Wire Line
-	4800 5650 5000 5650
-Connection ~ 4800 5650
-Wire Wire Line
 	5300 5650 5450 5650
 Wire Wire Line
@@
 Wire Wire Line
 	5450 6100 5450 6250
-Wire Wire Line
-	5450 6250 4800 6250
-Connection ~ 4800 6250
 Connection ~ 5450 5650
 $Comp
@@
 	4400 5300 5600 5300
 Wire Wire Line
-	4400 5650 4800 5650
-Wire Wire Line
 	6450 5300 6450 5000
 Connection ~ 3900 6250
@@
 Wire Wire Line
 	2950 1700 3200 1700
-Wire Wire Line
-	3500 1700 3950 1700
-Wire Wire Line
-	3950 1700 3950 2600
-Wire Wire Line
-	3950 2600 3200 2600
-Connection ~ 3200 2600
 $Comp
 L Device:R R7
@@
 	3000 4550 3250 4550
 Wire Wire Line
-	3550 4550 4000 4550
-Wire Wire Line
-	4000 4550 4000 5450
-Wire Wire Line
-	3200 5450 4000 5450
-Connection ~ 3200 5450
-Wire Wire Line
 	2800 5250 3000 5250
 $Comp
@@
 Connection ~ 2950 1700
 Wire Wire Line
-	3500 1200 3950 1200
-Wire Wire Line
-	3950 1200 3950 1700
-Connection ~ 3950 1700
+	3500 1200 3900 1200
 $Comp
 L Device:R R5
@@
 Wire Wire Line
 	3000 4050 3250 4050
-Wire Wire Line
-	3550 4050 4000 4050
-Wire Wire Line
-	4000 4050 4000 4550
 Connection ~ 3000 4550
-Connection ~ 4000 4550
 Text Notes 2500 1000 0    50   ~ 0
 Parallel resistor to change range of Rheostat
@@
 Wire Wire Line
 	6000 5300 6450 5300
+Wire Wire Line
+	3900 3400 5450 3400
+Wire Wire Line
+	4400 2800 5000 2800
+Wire Wire Line
+	4400 5650 5000 5650
+Wire Wire Line
+	3900 6250 5450 6250
+Wire Wire Line
+	3900 2800 3900 1700
+Wire Wire Line
+	3500 1700 3900 1700
+Connection ~ 3900 1700
+Wire Wire Line
+	3900 1700 3900 1200
+Wire Wire Line
+	3900 5650 3900 4550
+Wire Wire Line
+	3900 4550 3550 4550
+Wire Wire Line
+	3900 4550 3900 4050
+Wire Wire Line
+	3900 4050 3550 4050
+Connection ~ 3900 4550
 $EndSCHEMATC
