File: MCU.sch (KiCad schematic (older format))
At the start: 11 parts, among them J2 STLinkV2, SW1 SW_SPST, U13 STM32F051K4Tx

Commit message: corrected some psu errors
Connections:
- net +3V3: no longer DS1.2 (VDD), RV3.3
- new net +5V: DS1.2 (VDD), RV3.3
Other:
- moved on the sheet: C20, C21, C22, C23, C24, DS1, J2, R1, RV3, SW1, U13

Commit message: replaced capacitor multiplier by using a more powerful output transistor
Connections:
- net +3V3: no longer DS1.15 (LED(+))
- net +5V: now also DS1.15 (LED(+))
Changed lines of the file:
@@
 	-1   0    0    1
-$EndComp
-$Comp
-L power:+3V3 #PWR?
-U 1 1 600C20D0
-P 8900 2400
-AR Path="/604E5285/600C20D0" Ref="#PWR?"  Part="1"
-AR Path="/6096B205/600C20D0" Ref="#PWR?"  Part="1"
-AR Path="/604D4533/600C20D0" Ref="#PWR09"  Part="1"
-F 0 "#PWR09" H 8900 2250 50  0001 C CNN
-F 1 "+3V3" H 8915 2573 50  0000 C CNN
-F 2 "" H 8900 2400 50  0001 C CNN
-F 3 "" H 8900 2400 50  0001 C CNN
-	1    8900 2400
-	1    0    0    -1
 $EndComp
 Wire Wire Line
@@
 	1    0    0    -1
 $EndComp
+$Comp
+L power:+5V #PWR?
+U 1 1 60296553
+P 8900 2400
+F 0 "#PWR?" H 8900 2250 50  0001 C CNN
+F 1 "+5V" H 8915 2573 50  0000 C CNN
+F 2 "" H 8900 2400 50  0001 C CNN
+F 3 "" H 8900 2400 50  0001 C CNN
+	1    8900 2400
+	1    0    0    -1
+$EndComp
